Commit message: updated urdf and added gazebo plugins

File: src/nndrone_description/urdf/materials.xacro (robot description, xacro)
@@ -4,3 +4,9 @@
   <color rgba="0.700 0.700 0.700 1.000"/>
 </material>
+<material name="red">
+  <color rgba="1.00 0.0 0.00 1.000"/>
+</material>
+<material name="black">
+  <color rgba="0.10 0.10 0.100 1.000"/>
+</material>
 </robot>

File: src/nndrone_description/urdf/nndrone.xacro (robot description, xacro)
@@ -35,5 +35,5 @@
       <mesh filename="package://nndrone_description/meshes/prop_cw_1_1.stl" scale="0.001 0.001 0.001"/>
     </geometry>
-    <material name="silver"/>
+    <material name="red"/>
   </visual>
   <collision>
@@ -55,5 +55,5 @@
       <mesh filename="package://nndrone_description/meshes/prop_ccw_3_1.stl" scale="0.001 0.001 0.001"/>
     </geometry>
-    <material name="silver"/>
+    <material name="red"/>
   </visual>
   <collision>
@@ -75,5 +75,5 @@
       <mesh filename="package://nndrone_description/meshes/prop_cw_2_1.stl" scale="0.001 0.001 0.001"/>
     </geometry>
-    <material name="silver"/>
+    <material name="red"/>
   </visual>
   <collision>
@@ -95,5 +95,5 @@
       <mesh filename="package://nndrone_description/meshes/prop_ccw_4_1.stl" scale="0.001 0.001 0.001"/>
     </geometry>
-    <material name="silver"/>
+    <material name="red"/>
   </visual>
   <collision>
@@ -115,5 +115,5 @@
       <mesh filename="package://nndrone_description/meshes/lidar_1.stl" scale="0.001 0.001 0.001"/>
     </geometry>
-    <material name="silver"/>
+    <material name="black"/>
   </visual>
   <collision>
@@ -135,5 +135,5 @@
       <mesh filename="package://nndrone_description/meshes/pi_camera_1.stl" scale="0.001 0.001 0.001"/>
     </geometry>
-    <material name="silver"/>
+    <material name="black"/>
   </visual>
   <collision>

Commit message: fixed imu link and plugin configuration

File: src/nndrone_description/urdf/materials.xacro (robot description, xacro)
@@ -2,8 +2,11 @@
 <robot name="nndrone" xmlns:xacro="http://www.ros.org/wiki/xacro" >
 <material name="silver">
-  <color rgba="0.700 0.700 0.700 1.000"/>
+  <color rgba="0.900 0.900 0.900 1.000"/>
 </material>
 <material name="red">
   <color rgba="1.00 0.0 0.00 1.000"/>
+</material>
+<material name="yellow">
+  <color rgba="1.00 1.0 0.00 1.000"/>
 </material>
 <material name="black">

File: src/nndrone_description/urdf/nndrone.xacro (robot description, xacro)
@@ -8,6 +8,6 @@
     <inertial>
       <origin rpy="0 0 -1.5708" xyz="0.0 0.0 -0.055"/>
-      <mass value="0.5"/>
-      <inertia  ixx="0.0017350964305" ixy="0" ixz="0" iyy="0.00253016077525" iyz="0" izz="0.00365126915346" />
+      <mass value="1.0"/>
+      <inertia  ixx="0.00347019286099" ixy="0" ixz="0" iyy="0.0050603215505" iyz="0" izz="0.00730253830692" />
     </inertial>
     <visual>
@@ -21,7 +21,8 @@
       <origin rpy="0 0 -1.5708" xyz="0 0 -0.055"/>
       <geometry>
+        <!-- <box size="0.6 0.1 0.2"/> -->
         <mesh filename="package://nndrone_description/meshes/base_link.stl" scale="0.001 0.001 0.001"/>
       </geometry>
-      <surface>
+        <surface>
           <contact>
             <ode>
@@ -41,5 +42,5 @@
   <link name="prop_cw_1">
     <inertial>
-      <origin rpy="0 0 0" xyz="0.0 0.0 0.0"/>
+      <origin rpy="0 0 0" xyz="0.0 0.0 0.02"/>
       <mass value="0.027"/>
       <inertia  ixx="2.16576359834e-05" ixy="0" ixz="0" iyy="2.78597602888e-05" iyz="0" izz="4.9003356158e-05" />
@@ -50,56 +51,56 @@
         <mesh filename="package://nndrone_description/meshes/prop_cw_1_1.stl" scale="0.001 0.001 0.001"/>
       </geometry>
+      <material name="yellow"/>
+    </visual>
+    <collision>
+      <origin rpy="0 0 0" xyz="-0.0985 -0.0695 -0.055"/>
+      <geometry>
+        <mesh filename="package://nndrone_description/meshes/prop_cw_1_1.stl" scale="0.001 0.001 0.001"/>
+      </geometry>
+    </collision>
+  </link>
+  <link name="prop_ccw_3">
+    <inertial>
+      <origin rpy="0 0 0" xyz="0.0 0.0 0.02"/>
+      <mass value="0.027"/>
+      <inertia  ixx="2.16576359834e-05" ixy="0" ixz="0" iyy="2.78597602888e-05" iyz="0" izz="4.9003356158e-05" />
+    </inertial>
+    <visual>
+      <origin rpy="0 0 0" xyz="0.0985 -0.0695 -0.055"/>
+      <geometry>
+        <mesh filename="package://nndrone_description/meshes/prop_ccw_3_1.stl" scale="0.001 0.001 0.001"/>
+      </geometry>
+      <material name="yellow"/>
+    </visual>
+    <collision>
+      <origin rpy="0 0 0" xyz="0.0985 -0.0695 -0.055"/>
+      <geometry>
+        <mesh filename="package://nndrone_description/meshes/prop_ccw_3_1.stl" scale="0.001 0.001 0.001"/>
+      </geometry>
+    </collision>
+  </link>
+  <link name="prop_cw_2">
+    <inertial>
+      <origin rpy="0 0 0" xyz="0.0 0.0 0.02"/>
+      <mass value="0.027"/>
+      <inertia  ixx="2.16576359834e-05" ixy="0" ixz="0" iyy="2.78597602888e-05" iyz="0" izz="4.9003356158e-05" />
+    </inertial>
+    <visual>
+      <origin rpy="0 0 0" xyz="0.0985 0.0869 -0.055"/>
+      <geometry>
+        <mesh filename="package://nndrone_description/meshes/prop_cw_2_1.stl" scale="0.001 0.001 0.001"/>
+      </geometry>
       <material name="red"/>
     </visual>
     <collision>
-      <origin rpy="0 0 0" xyz="-0.0985 -0.0695 -0.055"/>
-      <geometry>
-        <mesh filename="package://nndrone_description/meshes/prop_cw_1_1.stl" scale="0.001 0.001 0.001"/>
-      </geometry>
-    </collision>
-  </link>
-  <link name="prop_ccw_3">
-    <inertial>
-      <origin rpy="0 0 0" xyz="0.0 0.0 0.0"/>
-      <mass value="0.027"/>
-      <inertia  ixx="2.16576359834e-05" ixy="0" ixz="0" iyy="2.78597602888e-05" iyz="0" izz="4.9003356158e-05" />
-    </inertial>
-    <visual>
-      <origin rpy="0 0 0" xyz="0.0985 -0.0695 -0.055"/>
-      <geometry>
-        <mesh filename="package://nndrone_description/meshes/prop_ccw_3_1.stl" scale="0.001 0.001 0.001"/>
-      </geometry>
-      <material name="red"/>
-    </visual>
-    <collision>
-      <origin rpy="0 0 0" xyz="0.0985 -0.0695 -0.055"/>
-      <geometry>
-        <mesh filename="package://nndrone_description/meshes/prop_ccw_3_1.stl" scale="0.001 0.001 0.001"/>
-      </geometry>
-    </collision>
-  </link>
-  <link name="prop_cw_2">
-    <inertial>
-      <origin rpy="0 0 0" xyz="0.0 0.0 0.0"/>
-      <mass value="0.027"/>
-      <inertia  ixx="2.16576359834e-05" ixy="0" ixz="0" iyy="2.78597602888e-05" iyz="0" izz="4.9003356158e-05" />
-    </inertial>
-    <visual>
       <origin rpy="0 0 0" xyz="0.0985 0.0869 -0.055"/>
       <geometry>
         <mesh filename="package://nndrone_description/meshes/prop_cw_2_1.stl" scale="0.001 0.001 0.001"/>
       </geometry>
-      <material name="red"/>
-    </visual>
-    <collision>
-      <origin rpy="0 0 0" xyz="0.0985 0.0869 -0.055"/>
-      <geometry>
-        <mesh filename="package://nndrone_description/meshes/prop_cw_2_1.stl" scale="0.001 0.001 0.001"/>
-      </geometry>
     </collision>
   </link>
   <link name="prop_ccw_4">
     <inertial>
-      <origin rpy="0 0 0" xyz="0.0 0.0 0.0"/>
+      <origin rpy="0 0 0" xyz="0.0 0.0 0.02"/>
       <mass value="0.027"/>
       <inertia  ixx="2.16576359834e-05" ixy="0" ixz="0" iyy="2.78597602888e-05" iyz="0" izz="4.9003356158e-05" />
@@ -151,13 +152,13 @@
         <origin rpy="0 0 0" xyz="0 0 0" />
         <mass value="0.15" />
-        <inertia  ixx="0.000520528929149" ixy="0" ixz="0" iyy="0.000759048232575" iyz="0" izz="0.00109538074604" />
+        <inertia  ixx="0.00001" ixy="0" ixz="0" iyy="0.00002" iyz="0" izz="0.00002" />
       </inertial>
-      <visual>
-      <origin rpy="0 0 0" xyz="0.0 -0.06725 -0.036"/>
-      <geometry>
-        <mesh filename="package://nndrone_description/meshes/imu.stl" scale="0.001 0.001 0.001"/>
-      </geometry>
-      <material name="black"/>
-      </visual>
+  </link>
+  <link name='gps_link'>
+    <inertial>
+      <origin rpy="0 0 0" xyz="0 0 0 " />
+      <mass value="0.15" />
+      <inertia ixx="0.00001" ixy="0.0" ixz="-0.0" iyy="0.00002" iyz="0.0" izz="0.00002" />
+    </inertial>
   </link>
   <joint name="Rev1" type="continuous">
@@ -195,6 +196,25 @@
     <child link="pi_camera_1"/>
   </joint>
-  <joint name="imu_joint" type="fixed">
-      <origin rpy="0 3.141593 0.0" xyz="0 0 0.0" />
+  <joint name="gps_joint" type="fixed">
+    <origin rpy="0 0 0" xyz="0 0 0" />
+    <parent link="base_link" />
+    <child link="gps_link" />
+  </joint>
+  <joint name="imu_joint" type="revolute">
+      <origin rpy="0 0 0" xyz="0 0 0"/>
+      <parent link="base_link" />
+      <child link="imu_link" />
+      <axis xyz="0 0 1"/>
+      <dynamics damping="1.0" friction="0.0"/>
+      <limit effort="0.0" lower="0.0" upper="0.0" velocity="0.0"/>
+      <!-- <use_parent_model_frame>0</use_parent_model_frame> -->
+<!--
+      <physics>
+        <ode>
+          <implicit_spring_damper>1</implicit_spring_damper>
+        </ode>
+      </physics>
+       -->
+      <!-- <origin rpy="0 0 0.0" xyz="0 0 0.0" />
       <parent link="base_link" />
       <child link="imu_link" />
@@ -204,5 +224,5 @@
           <implicit_spring_damper>1</implicit_spring_damper>
         </ode>
-      </physics>
+      </physics> -->
   </joint>
 </robot>
