Commit message: update description package

File: src/nndrone_description/urdf/nndrone.xacro (robot description, xacro)
@@ -7,10 +7,10 @@
   <link name="base_link">
     <inertial>
-      <origin rpy="0 0 0" xyz="6.920802996400466e-07 -0.006829490164314318 0.049664776612529236"/>
-      <mass value="0.1500"/>
-      <inertia ixx="0.004846" ixy="-0.0" ixz="-0.0" iyy="0.005607" iyz="-6.3e-05" izz="0.010017"/>
-    </inertial>
-    <visual>
-      <origin rpy="0 0 0" xyz="0 0 0"/>
+      <origin rpy="0 0 -1.5708" xyz="0.0 0.0 -0.055"/>
+      <mass value="0.5"/>
+      <inertia  ixx="0.0017350964305" ixy="0" ixz="0" iyy="0.00253016077525" iyz="0" izz="0.00365126915346" />
+    </inertial>
+    <visual>
+      <origin rpy="0 0 -1.5708" xyz="0 0 -0.055"/>
       <geometry>
         <mesh filename="package://nndrone_description/meshes/base_link.stl" scale="0.001 0.001 0.001"/>
@@ -19,8 +19,22 @@
     </visual>
     <collision>
-      <origin rpy="0 0 0" xyz="0 0 0"/>
+      <origin rpy="0 0 -1.5708" xyz="0 0 -0.055"/>
       <geometry>
         <mesh filename="package://nndrone_description/meshes/base_link.stl" scale="0.001 0.001 0.001"/>
       </geometry>
+      <surface>
+          <contact>
+            <ode>
+              <max_vel>100.0</max_vel>
+              <min_depth>0.001</min_depth>
+            </ode>
+          </contact>
+          <friction>
+            <ode>
+              <mu>1.0</mu>
+              <mu2>1.0</mu2>
+            </ode>
+          </friction>
+        </surface>
     </collision>
   </link>
@@ -29,5 +43,5 @@
       <origin rpy="0 0 0" xyz="0.0 0.0 0.0"/>
       <mass value="0.027"/>
-      <inertia ixx="1e-05" ixy="-0.0" ixz="0.0" iyy="1e-05" iyz="0.0" izz="2.1e-05"/>
+      <inertia  ixx="2.16576359834e-05" ixy="0" ixz="0" iyy="2.78597602888e-05" iyz="0" izz="4.9003356158e-05" />
     </inertial>
     <visual>
@@ -49,5 +63,5 @@
       <origin rpy="0 0 0" xyz="0.0 0.0 0.0"/>
       <mass value="0.027"/>
-      <inertia ixx="1e-05" ixy="0.0" ixz="-0.0" iyy="1e-05" iyz="0.0" izz="2.1e-05"/>
+      <inertia  ixx="2.16576359834e-05" ixy="0" ixz="0" iyy="2.78597602888e-05" iyz="0" izz="4.9003356158e-05" />
     </inertial>
     <visual>
@@ -69,5 +83,5 @@
       <origin rpy="0 0 0" xyz="0.0 0.0 0.0"/>
       <mass value="0.027"/>
-      <inertia ixx="1e-05" ixy="-0.0" ixz="-0.0" iyy="1e-05" iyz="-0.0" izz="2.1e-05"/>
+      <inertia  ixx="2.16576359834e-05" ixy="0" ixz="0" iyy="2.78597602888e-05" iyz="0" izz="4.9003356158e-05" />
     </inertial>
     <visual>
@@ -79,5 +93,5 @@
     </visual>
     <collision>
-      <origin rpy="0 0 0" xyz="0.0 0.0 0.0"/>
+      <origin rpy="0 0 0" xyz="0.0985 0.0869 -0.055"/>
       <geometry>
         <mesh filename="package://nndrone_description/meshes/prop_cw_2_1.stl" scale="0.001 0.001 0.001"/>
@@ -89,5 +103,5 @@
       <origin rpy="0 0 0" xyz="0.0 0.0 0.0"/>
       <mass value="0.027"/>
-      <inertia ixx="1e-05" ixy="0.0" ixz="0.0" iyy="1e-05" iyz="-0.0" izz="2.1e-05"/>
+      <inertia  ixx="2.16576359834e-05" ixy="0" ixz="0" iyy="2.78597602888e-05" iyz="0" izz="4.9003356158e-05" />
     </inertial>
     <visual>
@@ -118,10 +132,4 @@
       <material name="black"/>
     </visual>
-    <collision>
-      <origin rpy="0 0 0" xyz="-0.0 -0.077 -0.0415"/>
-      <geometry>
-        <mesh filename="package://nndrone_description/meshes/lidar_1.stl" scale="0.001 0.001 0.001"/>
-      </geometry>
-    </collision>
   </link>
   <link name="pi_camera_1">
@@ -138,56 +146,63 @@
       <material name="black"/>
     </visual>
-    <collision>
-      <origin rpy="0 0 0" xyz="0.0 -0.06725 -0.036"/>
-      <geometry>
-        <mesh filename="package://nndrone_description/meshes/pi_camera_1.stl" scale="0.001 0.001 0.001"/>
-      </geometry>
-    </collision>
   </link>
   <link name='imu_link'>
       <inertial>
         <origin rpy="0 0 0" xyz="0 0 0" />
-        <mass value="0.0051" />
-        <inertia ixx="0.059416" ixy="0.0" ixz="-0.0" iyy="0.066567" iyz="0.0" izz="0.059416" />
+        <mass value="0.15" />
+        <inertia  ixx="0.000520528929149" ixy="0" ixz="0" iyy="0.000759048232575" iyz="0" izz="0.00109538074604" />
       </inertial>
+      <visual>
+      <origin rpy="0 0 0" xyz="0.0 -0.06725 -0.036"/>
+      <geometry>
+        <mesh filename="package://nndrone_description/meshes/imu.stl" scale="0.001 0.001 0.001"/>
+      </geometry>
+      <material name="black"/>
+      </visual>
   </link>
   <joint name="Rev1" type="continuous">
-    <origin rpy="0 0 0" xyz="0.0985 0.0695 0.055"/>
+    <origin rpy="0 0 0" xyz="0.0695 -0.0985 0.001"/>
     <parent link="base_link"/>
     <child link="prop_cw_1"/>
-    <axis xyz="-0.0 0.0 1.0"/>
+    <axis xyz="0.0 0.0 1.0"/>
   </joint>
   <joint name="Rev3" type="continuous">
-    <origin rpy="0 0 0" xyz="-0.0985 0.0695 0.055"/>
+    <origin rpy="0 0 0" xyz="0.0695 0.0985 0.001"/>
     <parent link="base_link"/>
     <child link="prop_ccw_3"/>
-    <axis xyz="-0.0 0.0 1.0"/>
+    <axis xyz="0.0 0.0 1.0"/>
   </joint>
   <joint name="Rev2" type="continuous">
-    <origin rpy="0 0 0" xyz="-0.0985 -0.0869 0.055"/>
+    <origin rpy="0 0 0" xyz="-0.0869 0.0985 0.001"/>
     <parent link="base_link"/>
     <child link="prop_cw_2"/>
-    <axis xyz="-0.0 0.0 1.0"/>
+    <axis xyz="0.0 0.0 1.0"/>
   </joint>
   <joint name="Rev4" type="continuous">
-    <origin rpy="0 0 0" xyz="0.0985 -0.0869 0.055"/>
+    <origin rpy="0 0 0" xyz="-0.0869 -0.0985 0.001"/>
     <parent link="base_link"/>
     <child link="prop_ccw_4"/>
-    <axis xyz="-0.0 0.0 1.0"/>
-  </joint>
-  <joint name="Rigid5" type="fixed">
-    <origin rpy="0 0 0" xyz="0.0 0.077 0.0415"/>
+    <axis xyz="0.0 0.0 1.0"/>
+  </joint>
+  <joint name="lidar_joint" type="fixed">
+    <origin rpy="0 0 1.5708" xyz="0.077 0.0 -0.015"/>
     <parent link="base_link"/>
     <child link="lidar_1"/>
   </joint>
   <joint name="rpi_cam_joint" type="fixed">
-    <origin rpy="0 0 0" xyz="0.0 0.06725 0.036"/>
+    <origin rpy="0 0 0" xyz="0.06725 0.0 -0.020"/>
     <parent link="base_link"/>
     <child link="pi_camera_1"/>
   </joint>
   <joint name="imu_joint" type="fixed">
-      <origin rpy="0 3.141593 -1.5708" xyz="0 0 0" />
+      <origin rpy="0 3.141593 0.0" xyz="0 0 0.0" />
       <parent link="base_link" />
       <child link="imu_link" />
+      <dynamics damping="0.7"/>
+      <physics>
+        <ode>
+          <implicit_spring_damper>1</implicit_spring_damper>
+        </ode>
+      </physics>
   </joint>
 </robot>

Commit message: refine urdf

File: src/nndrone_description/urdf/nndrone.xacro (robot description, xacro)
@@ -5,6 +5,7 @@
   <xacro:include filename="$(find nndrone_description)/urdf/nndrone.gazebo" />
   <xacro:include filename="$(find nndrone_description)/urdf/plugins/plugins.gazebo" />
+  <xacro:include filename="$(find realsense_ros_gazebo)/xacro/tracker.xacro"/>
   <link name="base_link">
-    <inertial>
+     <inertial>
       <origin rpy="0 0 -1.5708" xyz="0.0 0.0 -0.055"/>
       <mass value="1.0"/>
@@ -21,21 +22,6 @@
       <origin rpy="0 0 -1.5708" xyz="0 0 -0.055"/>
       <geometry>
-        <!-- <box size="0.6 0.1 0.2"/> -->
-        <mesh filename="package://nndrone_description/meshes/base_link.stl" scale="0.001 0.001 0.001"/>
-      </geometry>
-        <surface>
-          <contact>
-            <ode>
-              <max_vel>100.0</max_vel>
-              <min_depth>0.001</min_depth>
-            </ode>
-          </contact>
-          <friction>
-            <ode>
-              <mu>1.0</mu>
-              <mu2>1.0</mu2>
-            </ode>
-          </friction>
-        </surface>
+          <box  size="0.15 0.15 0.05" />
+      </geometry>
     </collision>
   </link>
@@ -44,5 +30,5 @@
       <origin rpy="0 0 0" xyz="0.0 0.0 0.02"/>
       <mass value="0.027"/>
-      <inertia  ixx="2.16576359834e-05" ixy="0" ixz="0" iyy="2.78597602888e-05" iyz="0" izz="4.9003356158e-05" />
+      <inertia  ixx="2.78597602888e-05" ixy="0" ixz="0" iyy="2.78597602888e-05" iyz="0" izz="4.9003356158e-05" />
     </inertial>
     <visual>
@@ -64,5 +50,5 @@
       <origin rpy="0 0 0" xyz="0.0 0.0 0.02"/>
       <mass value="0.027"/>
-      <inertia  ixx="2.16576359834e-05" ixy="0" ixz="0" iyy="2.78597602888e-05" iyz="0" izz="4.9003356158e-05" />
+      <inertia  ixx="2.78597602888e-05" ixy="0" ixz="0" iyy="2.78597602888e-05" iyz="0" izz="4.9003356158e-05" />
     </inertial>
     <visual>
@@ -84,5 +70,5 @@
       <origin rpy="0 0 0" xyz="0.0 0.0 0.02"/>
       <mass value="0.027"/>
-      <inertia  ixx="2.16576359834e-05" ixy="0" ixz="0" iyy="2.78597602888e-05" iyz="0" izz="4.9003356158e-05" />
+      <inertia  ixx="2.78597602888e-05" ixy="0" ixz="0" iyy="2.78597602888e-05" iyz="0" izz="4.9003356158e-05" />
     </inertial>
     <visual>
@@ -104,5 +90,5 @@
       <origin rpy="0 0 0" xyz="0.0 0.0 0.02"/>
       <mass value="0.027"/>
-      <inertia  ixx="2.16576359834e-05" ixy="0" ixz="0" iyy="2.78597602888e-05" iyz="0" izz="4.9003356158e-05" />
+      <inertia  ixx="2.78597602888e-05" ixy="0" ixz="0" iyy="2.78597602888e-05" iyz="0" izz="4.9003356158e-05" />
     </inertial>
     <visual>
@@ -162,4 +148,7 @@
     </inertial>
   </link>
+ <xacro:realsense_T265 sensor_name="t_camera" parent_link="base_link" rate="30.0">
+  <origin rpy="0 0 0" xyz="0.1 0 0.0"/>
+</xacro:realsense_T265>
   <joint name="Rev1" type="continuous">
     <origin rpy="0 0 0" xyz="0.0695 -0.0985 0.001"/>
@@ -167,4 +156,5 @@
     <child link="prop_cw_1"/>
     <axis xyz="0.0 0.0 1.0"/>
+    <dynamics damping="0.005"/>
   </joint>
   <joint name="Rev3" type="continuous">
@@ -173,4 +163,5 @@
     <child link="prop_ccw_3"/>
     <axis xyz="0.0 0.0 1.0"/>
+    <dynamics damping="0.005"/>
   </joint>
   <joint name="Rev2" type="continuous">
@@ -179,4 +170,5 @@
     <child link="prop_cw_2"/>
     <axis xyz="0.0 0.0 1.0"/>
+    <dynamics damping="0.005"/>
   </joint>
   <joint name="Rev4" type="continuous">
@@ -185,4 +177,5 @@
     <child link="prop_ccw_4"/>
     <axis xyz="0.0 0.0 1.0"/>
+    <dynamics damping="0.005"/>
   </joint>
   <joint name="lidar_joint" type="fixed">

Commit message: fixed body jittering

File: src/nndrone_description/urdf/nndrone.xacro (robot description, xacro)
@@ -8,8 +8,8 @@
   <link name="base_link">
      <inertial>
-      <origin rpy="0 0 -1.5708" xyz="0.0 0.0 -0.055"/>
-      <mass value="1.0"/>
-      <inertia  ixx="0.00347019286099" ixy="0" ixz="0" iyy="0.0050603215505" iyz="0" izz="0.00730253830692" />
-    </inertial>
+        <origin rpy="0 0 0" xyz="0.0 0.0 -0.0"/>
+        <mass value="1.0"/>
+        <inertia  ixx="0.00347019286099" ixy="0" ixz="0" iyy="0.0050603215505" iyz="0" izz="0.00730253830692" />
+      </inertial>
     <visual>
       <origin rpy="0 0 -1.5708" xyz="0 0 -0.055"/>
@@ -20,7 +20,7 @@
     </visual>
     <collision>
-      <origin rpy="0 0 -1.5708" xyz="0 0 -0.055"/>
-      <geometry>
-          <box  size="0.15 0.15 0.05" />
+      <origin rpy="0 0 0" xyz="0 0 -0.0"/>
+      <geometry>
+          <box  size="0.18 0.2 0.1" />
       </geometry>
     </collision>
@@ -29,6 +29,6 @@
     <inertial>
       <origin rpy="0 0 0" xyz="0.0 0.0 0.02"/>
-      <mass value="0.027"/>
-      <inertia  ixx="2.78597602888e-05" ixy="0" ixz="0" iyy="2.78597602888e-05" iyz="0" izz="4.9003356158e-05" />
+      <mass value="0.025"/>
+      <inertia  ixx="9.75e-06" ixy="0" ixz="0" iyy="0.000166704" iyz="0" izz="0.000167604" />
     </inertial>
     <visual>
@@ -40,7 +40,8 @@
     </visual>
     <collision>
-      <origin rpy="0 0 0" xyz="-0.0985 -0.0695 -0.055"/>
-      <geometry>
-        <mesh filename="package://nndrone_description/meshes/prop_cw_1_1.stl" scale="0.001 0.001 0.001"/>
+      <origin rpy="0 0 0" xyz="0 0 0.02"/>
+      <geometry>
+        <cylinder radius="0.1" length="0.005"/>
+        <!-- <mesh filename="package://nndrone_description/meshes/prop_cw_1_1.stl" scale="0.001 0.001 0.001"/> -->
       </geometry>
     </collision>
@@ -49,6 +50,6 @@
     <inertial>
       <origin rpy="0 0 0" xyz="0.0 0.0 0.02"/>
-      <mass value="0.027"/>
-      <inertia  ixx="2.78597602888e-05" ixy="0" ixz="0" iyy="2.78597602888e-05" iyz="0" izz="4.9003356158e-05" />
+      <mass value="0.025"/>
+      <inertia  ixx="9.75e-06" ixy="0" ixz="0" iyy="0.000166704" iyz="0" izz="0.000167604" />
     </inertial>
     <visual>
@@ -60,7 +61,8 @@
     </visual>
     <collision>
-      <origin rpy="0 0 0" xyz="0.0985 -0.0695 -0.055"/>
-      <geometry>
-        <mesh filename="package://nndrone_description/meshes/prop_ccw_3_1.stl" scale="0.001 0.001 0.001"/>
+      <origin rpy="0 0 0" xyz="0 0 0.02"/>
+      <geometry>
+        <cylinder radius="0.1" length="0.005"/>
+        <!-- <mesh filename="package://nndrone_description/meshes/prop_ccw_3_1.stl" scale="0.001 0.001 0.001"/> -->
       </geometry>
     </collision>
@@ -69,8 +71,10 @@
     <inertial>
       <origin rpy="0 0 0" xyz="0.0 0.0 0.02"/>
-      <mass value="0.027"/>
-      <inertia  ixx="2.78597602888e-05" ixy="0" ixz="0" iyy="2.78597602888e-05" iyz="0" izz="4.9003356158e-05" />
-    </inertial>
-    <visual>
+      <mass value="0.025"/>
+      <inertia  ixx="9.75e-06" ixy="0" ixz="0" iyy="0.000166704" iyz="0" izz="0.000167604" />
+    </inertial>
+    <visual>
+    <collision>
+    </collision>>
       <origin rpy="0 0 0" xyz="0.0985 0.0869 -0.055"/>
       <geometry>
@@ -80,7 +84,8 @@
     </visual>
     <collision>
-      <origin rpy="0 0 0" xyz="0.0985 0.0869 -0.055"/>
-      <geometry>
-        <mesh filename="package://nndrone_description/meshes/prop_cw_2_1.stl" scale="0.001 0.001 0.001"/>
+      <origin rpy="0 0 0" xyz="0 0 0.02"/>
+      <geometry>
+        <cylinder radius="0.1" length="0.005"/>
+        <!-- <mesh filename="package://nndrone_description/meshes/prop_cw_2_1.stl" scale="0.001 0.001 0.001"/> -->
       </geometry>
     </collision>
@@ -89,6 +94,6 @@
     <inertial>
       <origin rpy="0 0 0" xyz="0.0 0.0 0.02"/>
-      <mass value="0.027"/>
-      <inertia  ixx="2.78597602888e-05" ixy="0" ixz="0" iyy="2.78597602888e-05" iyz="0" izz="4.9003356158e-05" />
+      <mass value="0.025"/>
+      <inertia  ixx="9.75e-06" ixy="0" ixz="0" iyy="0.000166704" iyz="0" izz="0.000167604" />
     </inertial>
     <visual>
@@ -100,7 +105,8 @@
     </visual>
     <collision>
-      <origin rpy="0 0 0" xyz="-0.0985 0.0869 -0.055"/>
-      <geometry>
-        <mesh filename="package://nndrone_description/meshes/prop_ccw_4_1.stl" scale="0.001 0.001 0.001"/>
+    <origin rpy="0 0 0" xyz="0 0 0.02"/>
+      <geometry>
+        <cylinder radius="0.1" length="0.005"/>
+        <!-- <mesh filename="package://nndrone_description/meshes/prop_ccw_4_1.stl" scale="0.001 0.001 0.001"/> -->
       </geometry>
     </collision>
@@ -122,5 +128,5 @@
   <link name="pi_camera_1">
     <inertial>
-      <origin rpy="0 0 0" xyz="-1.0210978849032173e-12 0.0 -0.004779083094555998"/>
+      <origin rpy="0 0 0" xyz="0 0 0"/>
       <mass value="0.01"/>
       <inertia ixx="0.0" ixy="0.0" ixz="0.0" iyy="0.0" iyz="-0.0" izz="0.0"/>
@@ -148,7 +154,42 @@
     </inertial>
   </link>
- <xacro:realsense_T265 sensor_name="t_camera" parent_link="base_link" rate="30.0">
+<!--
+  <xacro:realsense_T265 sensor_name="t_camera" parent_link="base_link" rate="30.0">
   <origin rpy="0 0 0" xyz="0.1 0 0.0"/>
-</xacro:realsense_T265>
+  </xacro:realsense_T265>
+-->
+ <joint name="Rev1" type="revolute">
+    <origin rpy="0 0 0" xyz="0.0695 -0.0985 0.001"/>
+    <parent link="base_link"/>
+    <child link="prop_cw_1"/>
+    <axis xyz="0 0 1"/>
+    <dynamics damping="0.004"/>
+    <limit lower="-1e+16" upper="1e+16" effort="5.0" velocity="2100"/>
+  </joint>
+  <joint name="Rev3" type="revolute">
+    <origin rpy="0 0 0" xyz="0.0695 0.0985 0.001"/>
+    <parent link="base_link"/>
+    <child link="prop_ccw_3"/>
+    <axis xyz="0 0 1"/>
+    <dynamics damping="0.004"/>
+    <limit lower="-1e+16" upper="1e+16" effort="5.0" velocity="2100"/>
+  </joint>
+  <joint name="Rev2" type="revolute">
+    <origin rpy="0 0 0" xyz="-0.0869 0.0985 0.001"/>
+    <parent link="base_link"/>
+    <child link="prop_cw_2"/>
+    <axis xyz="0 0 1"/>
+    <dynamics damping="0.004"/>
+    <limit lower="-1e+16" upper="1e+16" effort="5.0" velocity="2100"/>
+  </joint>
+  <joint name="Rev4" type="revolute">
+    <origin rpy="0 0 0" xyz="-0.0869 -0.0985 0.001"/>
+    <parent link="base_link"/>
+    <child link="prop_ccw_4"/>
+    <axis xyz="0 0 1"/>
+    <dynamics damping="0.004"/>
+    <limit lower="-1e+16" upper="1e+16" effort="5.0" velocity="2100"/>
+  </joint>
+<!--
   <joint name="Rev1" type="continuous">
     <origin rpy="0 0 0" xyz="0.0695 -0.0985 0.001"/>
@@ -156,5 +197,5 @@
     <child link="prop_cw_1"/>
     <axis xyz="0.0 0.0 1.0"/>
-    <dynamics damping="0.005"/>
+    <dynamics damping="0.004"/>
   </joint>
   <joint name="Rev3" type="continuous">
@@ -163,5 +204,5 @@
     <child link="prop_ccw_3"/>
     <axis xyz="0.0 0.0 1.0"/>
-    <dynamics damping="0.005"/>
+    <dynamics damping="0.004"/>
   </joint>
   <joint name="Rev2" type="continuous">
@@ -170,5 +211,5 @@
     <child link="prop_cw_2"/>
     <axis xyz="0.0 0.0 1.0"/>
-    <dynamics damping="0.005"/>
+    <dynamics damping="0.004"/>
   </joint>
   <joint name="Rev4" type="continuous">
@@ -177,6 +218,7 @@
     <child link="prop_ccw_4"/>
     <axis xyz="0.0 0.0 1.0"/>
-    <dynamics damping="0.005"/>
-  </joint>
+    <dynamics damping="0.004"/>
+  </joint>
+  -->
   <joint name="lidar_joint" type="fixed">
     <origin rpy="0 0 1.5708" xyz="0.077 0.0 -0.015"/>
@@ -201,21 +243,4 @@
       <dynamics damping="1.0" friction="0.0"/>
       <limit effort="0.0" lower="0.0" upper="0.0" velocity="0.0"/>
-      <!-- <use_parent_model_frame>0</use_parent_model_frame> -->
-<!--
-      <physics>
-        <ode>
-          <implicit_spring_damper>1</implicit_spring_damper>
-        </ode>
-      </physics>
-       -->
-      <!-- <origin rpy="0 0 0.0" xyz="0 0 0.0" />
-      <parent link="base_link" />
-      <child link="imu_link" />
-      <dynamics damping="0.7"/>
-      <physics>
-        <ode>
-          <implicit_spring_damper>1</implicit_spring_damper>
-        </ode>
-      </physics> -->
   </joint>
 </robot>

Commit message: added apriltag ros node

File: src/nndrone_description/urdf/nndrone.xacro (robot description, xacro)
@@ -227,5 +227,5 @@
   </joint>
   <joint name="rpi_cam_joint" type="fixed">
-    <origin rpy="0 0 0" xyz="0.06725 0.0 -0.020"/>
+    <origin rpy="0 1.57 0" xyz="0.06725 0.0 -0.020"/>
     <parent link="base_link"/>
     <child link="pi_camera_1"/>

Commit message: use standard box geometry

File: src/nndrone_description/urdf/nndrone.xacro (robot description, xacro)
@@ -7,5 +7,4 @@
   <xacro:include filename="$(find nndrone_description)/urdf/nndrone.gazebo" />
   <xacro:include filename="$(find nndrone_description)/urdf/plugins/plugins.gazebo" />
-  <xacro:include filename="$(find realsense_ros_gazebo)/xacro/tracker.xacro"/>
   <link name="base_link">
      <inertial>
@@ -24,4 +23,5 @@
       <origin rpy="0 0 0" xyz="0 0 -0.0"/>
       <geometry>
+        <!-- <mesh filename="package://nndrone_description/meshes/base_link.stl" scale="0.001 0.001 0.001"/> -->
           <box  size="0.18 0.2 0.1" />
       </geometry>
@@ -156,9 +156,4 @@
     </inertial>
   </link>
-<!--
-  <xacro:realsense_T265 sensor_name="t_camera" parent_link="base_link" rate="30.0">
-  <origin rpy="0 0 0" xyz="0.1 0 0.0"/>
-  </xacro:realsense_T265>
--->
  <joint name="Rev1" type="revolute">
     <origin rpy="0 0 0" xyz="0.0695 -0.0985 0.001"/>
@@ -193,34 +188,4 @@
     <limit lower="-1e+16" upper="1e+16" effort="5.0" velocity="2100"/>
   </joint>
-<!--
-  <joint name="Rev1" type="continuous">
-    <origin rpy="0 0 0" xyz="0.0695 -0.0985 0.001"/>
-    <parent link="base_link"/>
-    <child link="prop_cw_1"/>
-    <axis xyz="0.0 0.0 1.0"/>
-    <dynamics damping="0.004"/>
-  </joint>
-  <joint name="Rev3" type="continuous">
-    <origin rpy="0 0 0" xyz="0.0695 0.0985 0.001"/>
-    <parent link="base_link"/>
-    <child link="prop_ccw_3"/>
-    <axis xyz="0.0 0.0 1.0"/>
-    <dynamics damping="0.004"/>
-  </joint>
-  <joint name="Rev2" type="continuous">
-    <origin rpy="0 0 0" xyz="-0.0869 0.0985 0.001"/>
-    <parent link="base_link"/>
-    <child link="prop_cw_2"/>
-    <axis xyz="0.0 0.0 1.0"/>
-    <dynamics damping="0.004"/>
-  </joint>
-  <joint name="Rev4" type="continuous">
-    <origin rpy="0 0 0" xyz="-0.0869 -0.0985 0.001"/>
-    <parent link="base_link"/>
-    <child link="prop_ccw_4"/>
-    <axis xyz="0.0 0.0 1.0"/>
-    <dynamics damping="0.004"/>
-  </joint>
-  -->
   <joint name="lidar_joint" type="fixed">
     <origin rpy="0 0 1.5708" xyz="0.077 0.0 -0.015"/>
